File: PCB/attiny1616board1/attiny1616board1.kicad_pcb (KiCad board)
At the start: 2 copper layers, 100 x 60 mm, 62 parts, among them J1 5V_POWER, J10 SENSOR3_IN, J11 WS2813_OUT, J12 SERVO_OUT, J13 UPDI, J14 SERIAL, J15 SOLENOID1, J16 SOLENOID2, J2 5V_SERIES, J3 24V_POWER, J4 24V_SERIES, J5 CAN1, J6 CAN2, J7 ENABLE_TERMINATOR, J8 SENSOR1_IN, J9 SENSOR2_IN, Q1 S8050, Q2 S8550, Q3 AO3400A, Q4 S8050, Q5 S8550, Q6 AO3400A, SW1 SENSOR1_TEST, SW2 SENSOR2_TEST, SW3 SENSOR3_TEST, SW4 SW_DIP_x08, U1 ATtiny1616-S, U2 MCP2515-xSO, U3 MCP2562-E-P, Y1 16MHz

Commit message: 新7セグ・タイマー制御基板のデータを追加
Parts:
- added D3: 1N5819WS, Diode_SMD:D_SOD-323, F.Cu at (139.2, 81.0)
- added Q7: AO3401A, Package_TO_SOT_SMD:SOT-23, F.Cu at (125.2, 87.3)
- added R9: 10k, Resistor_SMD:R_0402_1005Metric, F.Cu at (123.3, 80.9)
- added SW5: RESET, MyLib:DTS-6-V-2, F.Cu at (118.2, 84.1)
- moved J13 30.2 mm to (145.6, 90.5)
- moved J14 12.9 mm to (132.2, 106.7), turned to -90 degrees
- moved J12 5.08 mm to (118.2, 74.6), turned to -90 degrees
- moved SW1 0.64 mm to (146.2, 82.2)
- moved SW2 0.64 mm to (158.9, 82.2)
- moved SW3 0.64 mm to (171.6, 82.2)
Connections:
- C1 pad 1: +5V -> VCC
- C2 pad 1: +5V -> VCC
- J13 pad 1: +5V -> Net-(D3-A)
- J13 pad 2: UPDI -> GND
- J13 pad 3: GND -> UPDI
- R1 pad 2: +5V -> VCC
- U1 pad 1: +5V -> VCC
- U1 pad 17: /MISO -> /MOSI
- U1 pad 18: /MOSI -> /MISO
- U2 pad 18: +5V -> VCC
- U3 pad 3: +5V -> VCC
Routing:
- net VCC: track 0.00 -> 90.0 mm, vias 0 -> 2
- net GND: track 102.9 -> 172.0 mm, vias 103 -> 97
- net +5V: track 247.4 -> 210.4 mm, vias 3 -> 2
- net Net-(Q7-G): track 0.00 -> 13.1 mm
- net Net-(D3-A): track 0.00 -> 11.1 mm, vias 0 -> 1
- net UPDI: track 24.6 -> 14.2 mm
- net LED_DI: track 34.7 -> 31.0 mm
- net TXD: track 10.3 -> 8.09 mm
- net /SS: track 56.1 -> 58.1 mm
- net /SCK: track 29.1 -> 31.0 mm, vias 0 -> 1
- net SV: track 34.2 -> 32.4 mm, vias 2 -> 1
- net /CAN_INT: track 26.1 -> 24.5 mm
- net RXD: track 9.74 -> 10.9 mm
- net /MISO: track 34.7 -> 33.7 mm, vias 1 -> 0
- net /MOSI: track 31.2 -> 30.6 mm, vias 1 -> 0
Other:
- board text added: "ATtiny1616 Solenoid Servo LED CAN Controller Rev. 2 2026/08 @daisuke_ym"
- board text added: "RESET"
- board text removed: "ATtiny1616 Solenoid Servo LED CAN Controller Rev. 1 2026/07 @daisuke_ym"
