File: PCB/attiny1616board1/attiny1616board1.kicad_sch (KiCad schematic)
At the start: 17 parts, among them J1 5V_POWER, J2 5V_SERIES, J3 24V_POWER, J4 24V_SERIES, J5 CAN1, J6 CAN2, J7 ENABLE_TERMINATOR, U1 ATtiny1616-S, U2 MCP2515-xSO, U3 MCP2562-E-P, Y1 16MHz

Commit message: 新7セグ・タイマー制御基板のデータを追加
Parts:
- added Q7: AO3401A, Package_TO_SOT_SMD:SOT-23, symbol Transistor_FET:AO3401A
- added R9: 10k, Resistor_SMD:R_0402_1005Metric, symbol Device:R
- added SW5: RESET, MyLib:DTS-6-V-2, symbol Switch:SW_DPST
Connections:
- net +5V: now also Q7.2 (S), SW5.1, SW5.3; no longer C1.1, C2.1, R1.2, U1.1 (VCC), U2.18 (VDD), U3.3 (VDD)
- net GND: now also R9.2
- net MISO: now also U1.18 (PA2); no longer U1.17 (PA1)
- net MOSI: now also U1.17 (PA1); no longer U1.18 (PA2)
- new net: Q7.1 (G), R9.1, SW5.2, SW5.4
- new net VCC: C1.1, C2.1, Q7.3 (D), R1.2, U1.1 (VCC), U2.18 (VDD), U3.3 (VDD)
Other:
- moved on the sheet: C1, C2, C3, C4, J1, J2, J3, J4, J5, J6, J7, R1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
